File: kicad-plan/desk-clock.kicad_pcb (KiCad board)
At the start: 2 copper layers, 80.5 x 52 mm, 10 parts, among them J2 1.8"TFT-screen-socket, M1 Motor_Servo

Commit message: Added new kicad plan
Parts:
- added J3: RTC-module, Connector_PinSocket_2.54mm:PinSocket_1x06_P2.54mm_Vertical, B.Cu at (167.0, 97.8)
- moved RV1 0.25 mm to (124.4, 63.6)
Connections:
- A1 pad 23: unconnected-(A1-A4-Pad23) -> Net-(A1-A4)
- A1 pad 24: unconnected-(A1-A5-Pad24) -> Net-(A1-A5)
- J2 pad 2: Net-(A1-D10) -> Net-(A1-D13)
- J2 pad 3: Net-(A1-D9) -> Net-(A1-D11)
- J2 pad 4: Net-(A1-D8) -> Net-(A1-D9)
- J2 pad 5: Net-(A1-D11) -> Net-(A1-D8)
- J2 pad 6: Net-(A1-D13) -> Net-(A1-D10)
- J2 pad 7: Net-(J2-Pin_7) -> Net-(BZ1--)
- J2 pad 8: Net-(BZ1--) -> Net-(J2-Pin_8)
- Toggle-switch1 pad 2: Net-(J2-Pin_7) -> Net-(J2-Pin_8)
Routing:
- net Net-(BZ1--): track 0.00 -> 214.1 mm, vias 0 -> 4
- net Net-(A1-+5V): track 1.70 -> 140.6 mm, vias 0 -> 4
- net Net-(A1-D10): track 0.00 -> 97.8 mm
- net Net-(A1-D8): track 0.00 -> 95.0 mm
- net Net-(A1-D9): track 0.00 -> 90.4 mm
- net (no net): track 0.00 -> 85.7 mm
- net Net-(A1-D6): track 0.00 -> 83.0 mm, vias 0 -> 1
- net Net-(A1-D13): track 0.00 -> 81.7 mm
- net Net-(A1-D11): track 0.00 -> 76.5 mm
- net Net-(A1-3V3): track 0.00 -> 76.0 mm
- net Net-(A1-A5): track 0.00 -> 71.4 mm, vias 0 -> 1
- net Net-(J2-Pin_8): track 0.00 -> 68.4 mm
- net Net-(A1-A4): track 0.00 -> 63.1 mm, vias 0 -> 1
- net Net-(A1-D4): track 0.00 -> 62.6 mm, vias 0 -> 1
- net Net-(A1-D7): track 0.00 -> 49.4 mm, vias 0 -> 1
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