File: kicad-plan/desk-clock.kicad_sch (KiCad schematic)
At the start: 10 parts, among them J2 1.8"TFT-screen-socket, M1 Motor_Servo

Commit message: Added new kicad plan
Parts:
- added J3: RTC-module, Connector_PinSocket_2.54mm:PinSocket_1x06_P2.54mm_Vertical, symbol Connector:Conn_01x06_Socket
Connections:
- net at A1.4 (GND), BZ1.2 (-), M1.3 (-)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: now also J2.7 (Pin_7), J3.6 (Pin_6); no longer J2.8 (Pin_8)
- net at J2.2 (Pin_2): now also A1.16 (D13); no longer A1.13 (D10)
- net at J2.3 (Pin_3): now also A1.14 (D11); no longer A1.12 (D9)
- net at J2.4 (Pin_4): now also A1.12 (D9); no longer A1.11 (D8)
- net at J2.5 (Pin_5): now also A1.11 (D8); no longer A1.14 (D11)
- net at J2.6 (Pin_6): now also A1.13 (D10); no longer A1.16 (D13)
- net at Toggle-switch1.2 (B): now also J2.8 (Pin_8); no longer J2.7 (Pin_7)
- net at A1.27 (+5V), M1.2 (+), RV1.3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: now also J3.5 (Pin_5)
- net at A1.23 (A4): now also J3.4 (Pin_4)
- net at A1.24 (A5): now also J3.3 (Pin_3)
